File: _autosave-IGEM_Device.kicad_pcb (KiCad board)
At the start: 2 copper layers, 50.2 x 47.6 mm, 28 parts, among them J1 67997-410HLF, J2 Electrode_Conn, J3 Batt_Conn, SW1 Power_Switch, U1 SaBLE-X-R2, U2 TC1014-2.85VCT713, U3 LMP91000SD_NOPB, U4 LM334MX_NOPB, U5 TPS79718QDCKRQ1, U6 G-NIMO-003

Commit message: PCB v1
Other:
- board size 50.2 x 47.6 mm -> 50.2 x 46.4 mm
Changed lines of the file:
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@@
   (gr_line (start 104.775 97.155) (end 104.775 90.17) (layer Edge.Cuts) (width 0.15))
   (gr_line (start 146.05 97.155) (end 104.775 97.155) (layer Edge.Cuts) (width 0.15))
-  (gr_line (start 146.05 88.9) (end 146.05 95.885) (layer Edge.Cuts) (width 0.15))
-  (gr_line (start 150.495 88.9) (end 146.05 88.9) (layer Edge.Cuts) (width 0.15))
+  (gr_line (start 146.05 90.17) (end 146.05 97.155) (layer Edge.Cuts) (width 0.15))
+  (gr_line (start 150.495 90.17) (end 146.05 90.17) (layer Edge.Cuts) (width 0.15))
   (gr_line (start 100.33 90.17) (end 100.33 50.8) (layer Edge.Cuts) (width 0.15))
   (gr_line (start 104.775 90.17) (end 100.33 90.17) (layer Edge.Cuts) (width 0.15))
-  (gr_line (start 150.495 49.53) (end 150.495 88.9) (layer Edge.Cuts) (width 0.15))
+  (gr_line (start 150.495 50.8) (end 150.495 90.17) (layer Edge.Cuts) (width 0.15))
   (gr_line (start 100.33 50.8) (end 150.495 50.8) (layer Edge.Cuts) (width 0.15))
   (via (at 110.49 74.295) (size 0.6) (drill 0.4) (layers F.Cu B.Cu) (net 4))

Commit message: Update to PCB and Gerber files
Parts:
- moved J2 1.91 mm to (125.1, 47.6)
- moved U3 1.91 mm to (125.1, 59.7)
- moved R1 1.42 mm to (144.8, 81.9)
- moved R2 1.42 mm to (141.6, 81.9)
- moved D1 1.27 mm to (137.2, 52.1)
- moved J3 1.27 mm to (109.9, 94.6)
- moved R5 0.64 mm to (135.9, 55.2)
- moved U4 0.64 mm to (145.4, 54.0)
- moved U1 0.64 mm to (131.4, 71.1)
- moved R3 0.63 mm to (138.4, 55.2)
Routing:
- net +2V85: track 99.5 -> 117.1 mm, vias 1 -> 3
- net /TEMP_OUT: track 29.3 -> 36.2 mm
- net +1V8: track 35.3 -> 30.8 mm
- net /EXT_TEMP_SCL: track 73.5 -> 69.7 mm
- net /IP_CONTROL: track 35.7 -> 37.5 mm
- net /JTAG_TDO: track 14.5 -> 12.9 mm
- net Net-(D1-PadA): track 6.65 -> 8.16 mm
- net +BATT: track 44.7 -> 45.7 mm
- net /EXT_TEMP_SDA: track 93.0 -> 92.1 mm
- net GND: track 212.3 -> 213.1 mm
- net /RESET: track 5.44 -> 6.08 mm
- net /JTAG_TMSC: track 4.17 -> 4.80 mm
- net /JTAG_TCXC: track 4.81 -> 5.44 mm
- net /POWER_GOOD: track 43.3 -> 44.0 mm
- net /IP_CATHODE: track 8.09 -> 8.71 mm
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Other:
- board size 50.2 x 46.4 mm -> 50.2 x 47 mm

Commit message: Minor changes
Other:
- rule via_min_size: 0.4 -> 0.5
